Commit message: a different launch file for ball_chaser + a smarter robot

File: my_robot/urdf/my_robot.xacro (robot description, xacro)
@@ -341,4 +341,6 @@
     <parent link = "left_leg_base"/>
     <axis xyz="0 1 0" rpy="0 0 0"/>
+    <limit effort="10000" velocity="1000"/>
+    <dynamics damping="0.5" friction="2.0"/>
   </joint>
   <joint type="continuous" name="right_wheel_back_hinge">
@@ -347,4 +349,6 @@
     <parent link = "right_leg_base"/>
     <axis xyz="0 1 0" rpy="0 0 0"/>
+    <limit effort="10000" velocity="1000"/>
+    <dynamics damping="0.5" friction="2.0"/>
   </joint>
   <joint type="fixed" name="camera_joint">

Commit message: robot finetuning

File: my_robot/urdf/my_robot.xacro (robot description, xacro)
@@ -342,5 +342,5 @@
     <axis xyz="0 1 0" rpy="0 0 0"/>
     <limit effort="10000" velocity="1000"/>
-    <dynamics damping="0.5" friction="2.0"/>
+    <dynamics damping="0.1" friction="0.5"/>
   </joint>
   <joint type="continuous" name="right_wheel_back_hinge">
@@ -350,5 +350,5 @@
     <axis xyz="0 1 0" rpy="0 0 0"/>
     <limit effort="10000" velocity="1000"/>
-    <dynamics damping="0.5" friction="2.0"/>
+    <dynamics damping="0.1" friction="0.5"/>
   </joint>
   <joint type="fixed" name="camera_joint">
